File: flat-nano/kicad/hp_sensor.kicad_sch (KiCad schematic)
At the start: 72 parts, among them J1 Hand-soldered cable (3 wires), J2 programming clip holes, J5 recovery clip holes (SWD), Q1 AO3400A, Q2 AO3400A, U1 R7FA4M1AB3CFM, U3 HT7550-1, U4 INA226, Y1 32.768kHz 12.5pF 3215

Commit message: Update flat-nano and hat to the reviewed designs; refresh the website
Boards (both at the Arduino Nano R4 outline, 43.18 x 17.78 mm):
- Hand-routed copper (preroute.py) replaces the auto-router; release.py
  rebuilds, checks (ERC, DRC all severities, parity, Kelvin, solder vias,
  layout quality) and exports the order files with a release manifest.
- Layout quality gate: power copper >= 0.5 mm outer / 1.2 mm inner,
  heat sources on the center line, mirrored side needles, left/right
  copper within 10% on every layer.
- flat-nano: 5 V buck regulator (LMR36503), single-sided assembly,
  cable solder holes, programming-clip holes. Hat: parts on both faces,
  Nano pins kept.
- R11 330 ohm -> 1.5 kohm so pin D4 stays within the RA4M1 4 mA limit.
- TH1 is the right needle and TH3 the left, as seen on the top face with
  the cable end up (pin map unchanged: A2 = TH1, A0 = TH3).
- No revision labels; old-version checksums and auto-router reports
  removed.

Website (docs/) and twin:
- Board data, drawing, current-flow lines, tags, parts list, guided tour
  and model match the current flat-nano.
- Plainer wording for the C3/C4 filtering explanations.

Co-Authored-By: Claude Opus 5.5 <noreply@anthropic.com>
Parts:
- removed C5, C6: 18p, Capacitor_SMD:C_0402_1005Metric, symbol Device:C
- removed J5: recovery clip holes (SWD), hp_sensor:ClipRow_1x05_P2.54mm, symbol Connector_Generic:Conn_01x05
- removed Q2: AO3400A, Package_TO_SOT_SMD:SOT-23, symbol Transistor_FET:AO3400A
- removed R12: 1.5k, Resistor_SMD:R_0402_1005Metric, symbol Device:R
- removed R17: 100k, Resistor_SMD:R_0402_1005Metric, symbol Device:R
- removed U3: HT7550-1, Package_TO_SOT_SMD:SOT-89-3, symbol Regulator_Linear:HT75xx-1-SOT89
- removed Y1: 32.768kHz 12.5pF 3215, Crystal:Crystal_SMD_3215-2Pin_3.2x1.5mm, symbol Device:Crystal
- added C18: 100n 50V, Capacitor_SMD:C_0402_1005Metric, symbol Device:C
- added C19: 100n, Capacitor_SMD:C_0402_1005Metric, symbol Device:C
- added C20: 1u, Capacitor_SMD:C_0402_1005Metric, symbol Device:C
- added C3: 22u 25V, Capacitor_SMD:C_1206_3216Metric, symbol Device:C
- added L1: 22uH, Inductor_SMD:L_Sunlord_SWPA4020S, symbol Device:L
- added U3: LMR36503R5RPER, hp_sensor:TI_RPE0009A_VQFN-HR-9_2x2mm, symbol hp_sensor:LMR36503R5
- C1: Note (none) -> buck input capacitor (datasheet minimum 4.7 uF)
- C17: value 10u 10V -> 10u 25V
- C2: value 10u 10V -> 22u 25V; footprint Capacitor_SMD:C_0805_2012Metric -> Capacitor_SMD:C_1206_3216Metric; Note (none) -> buck output capacitor (22 uF rated)
- D1, D5, D7: value 1A 40V Schottky (SOD-123F) -> 1A 40V Schottky (SOD-323); footprint Diode_SMD:D_SOD-123F -> Diode_SMD:D_SOD-323
- J1: Note 1 = 12V, 2 = SDI-12 data, 3 = GND; hand-solder after assemb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 -> 1 = 12V (center hole, square), 2 = SDI-12 data, 3 = GND; ha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
- R11: value 10 -> 1.5k; Note filters the reference node -> limits pin D4 (RA4M1 P103) to 3.3 mA while C13 charges; the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
- TH1: Note left prong -> right prong
- TH3: Note right prong -> left prong
Connections:
- net TH_RTN is gone; now on net GND: TH1.2, TH2.2, TH3.2, TH4.2
- net +5V: no longer R11.1
- net D4_EXC: now also R11.1
- net GND: now also C18.2, C20.2, C3.2, U3.1 (RT), U3.9 (GND)
- net VIN_P: now also C18.1, C3.1, U3.3 (EN), U3.4 (VIN)
- net 5V_LDO renamed 5V_BUCK
- net 5V_BUCK: now also L1.2, U3.8 (VOUT)
- net A0_TH1 renamed A2_TH1
- net A2_TH1: now also U1.63 (P001/AN001); no longer U1.53 (P014/AN009)
- net A2_TH3 renamed A0_TH3
- net A0_TH3: now also U1.53 (P014/AN009); no longer U1.63 (P001/AN001)
- net SWCLK: no longer names the net of U1.32 (P300/SWCLK)
- net SWDIO: no longer names the net of U1.33 (P108/SWDIO)
- net XCIN: no longer names the net of U1.6 (P215/XCIN)
- net XCOUT: no longer names the net of U1.7 (P214/XCOUT)
- new net BOOT: C19.1, U3.6 (BOOT)
- new net SW: C19.2, L1.1, U3.5 (SW)
- new net VCC_BUCK: C20.1, U3.7 (VCC)
- no-connect marks 33 -> 38
Other:
- note added: "FIRMWARE ACCESS (no soldering) - J2 is a row of five holes for an off-the-shelf 2.54 mm 5-pin pogo clip. Holes 1-4 carry USB (5V, D-, D+, GND): plug a 'USB to 4-pin Dupont' cable onto the clip and the board is an 'Arduino UNO R4 Minima' in the IDE. Hole 5 = BOOT: only for the very first load of the Arduino bootloader, put a jumper cap across clip pins 4-5 while plugging in. Recovery never needs a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"
- note added: "HEATER RESISTOR CHAIN (top of center prong) - 17 x 3.3 ohm 1% 0603 in series, 2.6 mm pitch. EXACT Vishay CRCW06033R30FKEAHP, 0.33 W at 70 C; no ordinary 0.1 W substitutes. Return is on bottom copper. Nominal full-ON power 2.34 W at 12 V, 3.41 W at 14.4 V with specified cable losses. PWM controls average energy; instantaneous ratings still apply. Qualify the potted needle thermally."
- note added: "HP-SDI12-NANO / COMPACT FLAT - 11.5-14.4 V battery supply over the 3-wire SDI-12 cable. J1 has three bare cable solder holes (VIN, data, ground); no connector is fitted. 5 V comes from a buck converter (TI LMR36503R5, 5 V fixed, ~4 uA no-load, 2.2 MHz with RT tied to GND), which wastes several times less heat than a linear regulator."
- note added: "MICROCONTROLLER - Renesas RA4M1 (R7FA4M1AB3CFM), the Arduino UNO R4 / Nano R4 chip, wired exactly like the UNO R4 Minima so the stock board package and Arduino pin names apply (nets D2, D4, D9, A0-A5). Runs at 5 V. Support circuit (NMI, USB sense, VCC_USB, VCL) follows Arduino's Nano R4 schematic. No 32.768 kHz crystal: the stock Arduino core clocks the CPU and USB from the internal HOCO and the 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"
- note added: "THERMISTORS - pin map (same on flat-nano and hat): A2 = TH1 right needle, A1 = TH2 heater-needle tip, A0 = TH3 left needle, A3 = TH4 board body (left/right seen on the top face, cable end up, needles down). Required firmware: 14-bit ADC, external VREF (AR_EXTERNAL), 64 readings averaged; actual noise and accuracy require measurement. The dividers and ADC reference share VREF. D4 powers the divide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"
- note removed: "FIRMWARE ACCESS (no soldering) - J2 is a row of five holes for an off-the-shelf 2.54 mm 5-pin pogo clip. Holes 1-4 carry USB (5V, D-, D+, GND): plug a 'USB to 4-pin Dupont' cable onto the clip and the board is an 'Arduino UNO R4 Minima' in the IDE. Hole 5 = BOOT: only for the very first load of the Arduino bootloader, put a jumper cap across clip pins 4-5 while plugging in. J5 = a second five-hol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"
- note removed: "HEATER RESISTOR CHAIN (top of centre prong) - 17 x 3.3 ohm 1% 0603 in series, 2.6 mm pitch. EXACT Vishay CRCW06033R30FKEAHP, 0.33 W at 70 C; no ordinary 0.1 W substitutes. Return is on bottom copper. Nominal full-ON power 2.34 W at 12 V, 3.41 W at 14.4 V with specified cable losses. PWM controls average energy; instantaneous ratings still apply. Qualify the potted needle thermally."
- note removed: "HP-SDI12-NANO r2 / COMPACT FLAT - 11.5-14.4 V battery supply over the 3-wire SDI-12 cable. J1 has three bare cable solder holes (VIN, data, ground); no connector is fitted. Asleep the board draws only the regulator (2.5 uA) plus MCU standby current."
- note removed: "MICROCONTROLLER - Renesas RA4M1 (R7FA4M1AB3CFM), the Arduino UNO R4 / Nano R4 chip, wired exactly like the UNO R4 Minima so the stock board package and Arduino pin names apply (nets D2, D4, D9, A0-A5). Runs at 5 V. Support circuit (NMI, USB sense, VCC_USB, VCL) follows Arduino's Nano R4 schematic."
- note removed: "THERMISTORS - required firmware: 14-bit ADC, external VREF (AR_EXTERNAL), 64 readings averaged; actual noise and accuracy require measurement. The dividers and ADC reference share VREF. D4 switches thermistor ground through Q2 to reduce self-heating. Sequence: D4 HIGH, wait 10 ms, read, D4 LOW. R_ntc = Rref * code / (full scale - code). NTC = Murata NCP15XH103F03RC (10k, 1%); Rref = 10k 0.1% 25 p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"
- title: Compact heat-pulse soil sensor, SDI-12 (HP-SDI12-NANO r2) -> Compact heat-pulse soil sensor, SDI-12 (HP-SDI12-NANO)

Commit message: Prefer JLC Basic/Preferred parts and fewer BOM lines; wider primer page
Flat-nano 27 -> 25 BOM lines (13 -> 9 Extended), hat 21 -> 20 (10 -> 6):
- Schottky diodes: 1N5819WS C191023 (Basic, same SOD-323)
- C1 and C17: one 10 uF 50 V 0805 part, C440198 (Basic)
- all 100 nF: the 50 V part C307331 (Basic)
- C4 3.3 nF: C26404 (Preferred); SMF16CA/SMF15CA TVS: C19077511/C19077510 (Preferred)
Copper and placement unchanged (all tracks, vias and positions identical); full
release checks pass. Twin parts data, flat-nano README and primer Appendix A
updated to match.

Primer page: wider column, larger text and more space between sections on
screen; print layout unchanged.

Co-Authored-By: Claude Opus 5.5 <noreply@anthropic.com>
Parts:
- C1: value 4.7u 50V -> 10u 50V
- C17: value 10u 25V -> 10u 50V
- C18: value 100n 50V -> 100n
