File: hat/kicad/hp_hat.kicad_sch (KiCad schematic)
At the start: 54 parts, among them J1 Hand-soldered cable (3 wires), J3 Nano solder-stack header, J4 Nano solder-stack header, Q1 AO3400A, Q2 AO3400A, U4 INA226

Commit message: Update flat-nano and hat to the reviewed designs; refresh the website
Boards (both at the Arduino Nano R4 outline, 43.18 x 17.78 mm):
- Hand-routed copper (preroute.py) replaces the auto-router; release.py
  rebuilds, checks (ERC, DRC all severities, parity, Kelvin, solder vias,
  layout quality) and exports the order files with a release manifest.
- Layout quality gate: power copper >= 0.5 mm outer / 1.2 mm inner,
  heat sources on the center line, mirrored side needles, left/right
  copper within 10% on every layer.
- flat-nano: 5 V buck regulator (LMR36503), single-sided assembly,
  cable solder holes, programming-clip holes. Hat: parts on both faces,
  Nano pins kept.
- R11 330 ohm -> 1.5 kohm so pin D4 stays within the RA4M1 4 mA limit.
- TH1 is the right needle and TH3 the left, as seen on the top face with
  the cable end up (pin map unchanged: A2 = TH1, A0 = TH3).
- No revision labels; old-version checksums and auto-router reports
  removed.

Website (docs/) and twin:
- Board data, drawing, current-flow lines, tags, parts list, guided tour
  and model match the current flat-nano.
- Plainer wording for the C3/C4 filtering explanations.

Co-Authored-By: Claude Opus 5.5 <noreply@anthropic.com>
Parts:
- removed C2: 10u 10V, Capacitor_SMD:C_0805_2012Metric, symbol Device:C
- removed Q2: AO3400A, Package_TO_SOT_SMD:SOT-23, symbol Transistor_FET:AO3400A
- removed R12: 1.5k, Resistor_SMD:R_0402_1005Metric, symbol Device:R
- removed R17: 100k, Resistor_SMD:R_0402_1005Metric, symbol Device:R
- added C17: 10u 25V, Capacitor_SMD:C_0805_2012Metric, symbol Device:C
- added C3: 22u 25V, Capacitor_SMD:C_1206_3216Metric, symbol Device:C
- D1: value 1A 40V Schottky (SOD-123F) -> 1A 40V Schottky (SOD-323); footprint Diode_SMD:D_SOD-123F -> Diode_SMD:D_SOD-323
- J1: footprint hp_sensor:CablePads_1x03_P4mm -> hp_sensor:CableSolder_1x03
- R11: value 10 -> 1.5k; Note filters the reference node -> limits pin D4 (RA4M1 P103) to 3.3 mA while C13 charges; the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
- TH1: Note left prong -> right prong
- TH3: Note right prong -> left prong
Connections:
- net TH_RTN is gone; now on net GND: TH1.2, TH2.2, TH3.2, TH4.2
- net +5V: now also C17.1; no longer R11.1
- net D4_EXC: now also R11.1
- net GND: now also C17.2, C3.2
- net VIN_P: now also C3.1
- net A0_TH1 renamed A2_TH1
- net A2_TH1: now also J4.6 (Pin_6); no longer J4.4 (Pin_4)
- net A2_TH3 renamed A0_TH3
- net A0_TH3: now also J4.4 (Pin_4); no longer J4.6 (Pin_6)
Other:
- note added: "HEATER RESISTOR CHAIN (top side of the center prong only) - 17 x 3.3 ohm 1% 0603 in series, 2.6 mm pitch. EXACT Vishay CRCW06033R30FKEAHP, 0.33 W at 70 C. The return runs on the bottom copper of the prong. Use Panasonic ERJ2GEJ5R1X, 0.1 W; resistor tolerance and local temperature affect the margin. First resistor starts outside the epoxy body. Firmware must detect zero heater current as a fault."
- note added: "THERMISTORS - pin map (same as flat-nano): A2 = TH1 right needle, A1 = TH2 heater-needle tip, A0 = TH3 left needle, A3 = TH4 board body (left/right seen on the top face, toward the Nano, cable end up, needles down; from the outer face they appear swapped). Dividers and Nano AREF share VREF. D4 powers them through R11, so they are off between readings (no self-heating) and the reading stays ratiom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"
- note removed: "HEATER RESISTOR CHAIN (top side of the centre prong only) - 17 x 3.3 ohm 1% 0603 in series, 2.6 mm pitch. EXACT Vishay CRCW06033R30FKEAHP, 0.33 W at 70 C. The return runs on the bottom copper of the prong. Use Panasonic ERJ2GEJ5R1X, 0.1 W; resistor tolerance and local temperature affect the margin. First resistor starts outside the epoxy body. Firmware must detect zero heater current as a fault."
- note removed: "THERMISTORS - dividers and Nano AREF share filtered VREF. Q2 switches their ground return to reduce self-heating between readings. Firmware: analogReference(AR_EXTERNAL), analogReadResolution(14); D4 HIGH, wait 10 ms, sample, D4 LOW. Verify settling, noise and calibration on assembled hardware. NTC = Murata NCP15XH103F03RC (10k, 1%); Rref = 10k 0.1% 25 ppm."
- title: Compact heat-pulse hat for Arduino Nano R4, SDI-12 (rev 4) -> Compact heat-pulse hat for Arduino Nano R4, SDI-12

Commit message: Prefer JLC Basic/Preferred parts and fewer BOM lines; wider primer page
Flat-nano 27 -> 25 BOM lines (13 -> 9 Extended), hat 21 -> 20 (10 -> 6):
- Schottky diodes: 1N5819WS C191023 (Basic, same SOD-323)
- C1 and C17: one 10 uF 50 V 0805 part, C440198 (Basic)
- all 100 nF: the 50 V part C307331 (Basic)
- C4 3.3 nF: C26404 (Preferred); SMF16CA/SMF15CA TVS: C19077511/C19077510 (Preferred)
Copper and placement unchanged (all tracks, vias and positions identical); full
release checks pass. Twin parts data, flat-nano README and primer Appendix A
updated to match.

Primer page: wider column, larger text and more space between sections on
screen; print layout unchanged.

Co-Authored-By: Claude Opus 5.5 <noreply@anthropic.com>
Parts:
- C1: value 4.7u 50V -> 10u 50V
- C17: value 10u 25V -> 10u 50V
